Commit message: Update urdf file

File: application/src/al5d_description/urdf/al5d.urdf (robot description, URDF)
Before this commit: robot lynxmotion_arm, 8 links, 7 joints
Links:
- link base_link: mass 1 -> None; geometry visual cylinder length=0.04 radius=0.095
- link forearm: mass 0.4 -> None; geometry visual cylinder length=0.20 radius=0.015
- link gripper_left: mass 0.1 -> None; geometry visual box size=0.02 0.02 0.03
- link gripper_right: mass 0.1 -> None; geometry visual box size=0.02 0.02 0.03
- link hand: mass 0.1 -> None; geometry visual box size=0.02 0.07 0.025
- link turret: mass 1 -> None; geometry visual cylinder length=0.005 radius=0.095
- link upperarm: mass 0.6 -> None; geometry visual box size=0.02 0.08 0.18
- link wrist: mass 0.4 -> None; geometry visual box size=0.02 0.05 0.06
